Commit message: add launch xml

File: minibot_description/urdf/minibot_ros2_control_gazebo.urdf.xacro (robot description, xacro)
@@ -1,5 +1,5 @@
 <?xml version="1.0"?>
 <robot xmlns:xacro="http://www.ros.org/wiki/xacro">
-    <xacro:macro name="insert_ros2_control" params="prefix is_sim:=^|false robot_port_name robot_baudrate">
+    <xacro:macro name="insert_ros2_control" params="prefix is_sim:=^|true robot_port_name robot_baudrate">
         <ros2_control name="${prefix}minibot_system" type="system">
             <hardware>

File: minibot_description/urdf/robot_gazebo.urdf.xacro (robot description, xacro)
@@ -6,5 +6,5 @@
     <xacro:include filename="$(find minibot_description)/urdf/minibot_ros2_control.urdf.xacro"/>
     <xacro:arg name="prefix" default=""/>
-    <xacro:arg name="is_sim" default="false"/>
+    <xacro:arg name="is_sim" default="true"/>
     <xacro:arg name="robot_port_name" default="/dev/ttyArduino"/>
     <xacro:arg name="robot_baudrate" default="500000"/>
