Commit message: model load in urdf fix (package -> file)

File: minibot_description/urdf/minibot.urdf.xacro (robot description, xacro)
@@ -9,5 +9,5 @@
                 <origin xyz="0 0 0" rpy="0 0 0"/>
                 <geometry>
-                    <mesh filename="package://minibot_description/meshes/visual/base_link.dae" scale="1 1 1"/>
+                    <mesh filename="file://$(find minibot_description)/meshes/visual/base_link.dae" scale="1 1 1"/>
                 </geometry>
             </visual>
@@ -15,5 +15,5 @@
                 <origin xyz="0 0 0" rpy="0 0 0"/>
                 <geometry>
-                    <mesh filename="package://minibot_description/meshes/collision/base_link.stl" scale="1 1 1"/>
+                    <mesh filename="file://$(find minibot_description)/meshes/collision/base_link.stl" scale="1 1 1"/>
                 </geometry>
             </collision>
@@ -35,5 +35,5 @@
                     <origin xyz="0 0 0" rpy="0 0 ${dir * pi/2}"/>
                     <geometry>
-                        <mesh filename="package://minibot_description/meshes/visual/wheel.dae" scale="1 1 1"/>
+                        <mesh filename="file://$(find minibot_description)/meshes/visual/wheel.dae" scale="1 1 1"/>
                     </geometry>
                 </visual>
@@ -41,5 +41,5 @@
                     <origin xyz="0 0 0" rpy="0 0 ${dir * pi/2}"/>
                     <geometry>
-                        <mesh filename="package://minibot_description/meshes/collision/wheel.stl" scale="1 1 1"/>
+                        <mesh filename="file://$(find minibot_description)/meshes/collision/wheel.stl" scale="1 1 1"/>
                     </geometry>
                 </collision>
@@ -65,5 +65,5 @@
                 <origin xyz="0 0 0" rpy="0 0 0"/>
                 <geometry>
-                    <mesh filename="package://minibot_description/meshes/visual/front_camera.dae" scale="1 1 1"/>
+                    <mesh filename="file://$(find minibot_description)/meshes/visual/front_camera.dae" scale="1 1 1"/>
                 </geometry>
             </visual>
@@ -71,5 +71,5 @@
                 <origin xyz="0 0 0" rpy="0 0 0"/>
                 <geometry>
-                    <mesh filename="package://minibot_description/meshes/collision/front_camera.stl" scale="1 1 1"/>
+                    <mesh filename="file://$(find minibot_description)/meshes/collision/front_camera.stl" scale="1 1 1"/>
                 </geometry>
             </collision>
@@ -95,5 +95,5 @@
                 <origin xyz="0 0 0" rpy="0 0 0"/>
                 <geometry>
-                    <mesh filename="package://minibot_description/meshes/visual/ul_sensor.dae" scale="1 1 1"/>
+                    <mesh filename="file://$(find minibot_description)/meshes/visual/ul_sensor.dae" scale="1 1 1"/>
                 </geometry>
             </visual>
@@ -101,5 +101,5 @@
                 <origin xyz="0 0 0" rpy="0 0 0"/>
                 <geometry>
-                    <mesh filename="package://minibot_description/meshes/collision/ul_sensor.stl" scale="1 1 1"/>
+                    <mesh filename="file://$(find minibot_description)/meshes/collision/ul_sensor.stl" scale="1 1 1"/>
                 </geometry>
             </collision>

File: minibot_description/urdf/minibot_gazebo.urdf.xacro (robot description, xacro)
@@ -16,5 +16,4 @@
             <kp>10000000.0</kp>
             <kd>1.0</kd>
-            <!-- <minDepth>0.001</minDepth> -->
         </gazebo>
         <gazebo reference="${prefix}r_wheel">
@@ -23,29 +22,27 @@
             <kp>10000000.0</kp>
             <kd>1.0</kd>
-            <!-- <minDepth>0.001</minDepth> -->
         </gazebo>
         <gazebo reference="${prefix}base_link">
             <mu1>0.0</mu1>
             <mu2>0.0</mu2>
-            <!-- <minDepth>0.001</minDepth> -->
         </gazebo>
-        <gazebo reference="${prefix}laser_link">
+        <gazebo reference="laser_link">
             <sensor name="laser" type="ray">
                 <pose>0 0 0 0 0 0</pose>
-                <always_on>1</always_on>
-                <update_rate>15</update_rate>
+                <always_on>true</always_on>
+                <update_rate>5</update_rate>
                 <visualize>false</visualize>
                 <ray>
                     <scan>
                         <horizontal>
-                            <samples>375</samples>
+                            <samples>180</samples>
                             <resolution>1</resolution>
-                            <min_angle>${-180*pi/180}</min_angle>
-                            <max_angle>${180*pi/180}</max_angle>
+                            <min_angle>-3.14159</min_angle>
+                            <max_angle>3.14159</max_angle>
                         </horizontal>
                     </scan>
                     <range>
                         <min>0.12</min>
-                        <max>8.0</max>
+                        <max>6.0</max>
                         <resolution>0.05</resolution>
                     </range>
@@ -60,5 +57,4 @@
                         <remapping>~/out:=scan</remapping>
                     </ros>
-                    <frame_name>${prefix}laser_link</frame_name>
                     <output_type>sensor_msgs/LaserScan</output_type>
                 </plugin>
@@ -88,7 +84,7 @@
                 <plugin name="${prefix}camera_controller" filename="libgazebo_ros_camera.so">
                     <ros>
-                        <!-- <namespace>${prefix}camera</namespace> -->
-                        <!-- <remapping>camera1/image_raw:=camera/image_test</remapping>
-                        <remapping>camera_info:=camera_info_test</remapping> -->
+                        <namespace>${prefix}camera</namespace>
+                        <remapping>camera1/image_raw:=camera/image_test</remapping>
+                        <remapping>camera_info:=camera_info_test</remapping>
                     </ros>
                     <frame_name>camera_link</frame_name>

File: minibot_description/urdf/robot.urdf.xacro (robot description, xacro)
@@ -18,5 +18,5 @@
             <origin xyz="0 0 0" rpy="0 0 0"/>
             <geometry>
-                <mesh filename="package://minibot_description/meshes/visual/ydlidar_x2_assy.dae" scale="1 1 1"/>
+                <mesh filename="file://$(find minibot_description)/meshes/visual/ydlidar_x2_assy.dae" scale="1 1 1"/>
             </geometry>
         </visual>
@@ -24,5 +24,5 @@
             <origin xyz="0 0 0" rpy="0 0 0"/>
             <geometry>
-                <mesh filename="package://minibot_description/meshes/collision/ydlidar_x2_assy.stl" scale="1 1 1"/>
+                <mesh filename="file://$(find minibot_description)/meshes/collision/ydlidar_x2_assy.stl" scale="1 1 1"/>
             </geometry>
         </collision>

File: minibot_description/urdf/robot_gazebo.urdf.xacro (robot description, xacro)
@@ -19,5 +19,5 @@
             <origin xyz="0 0 0" rpy="0 0 0"/>
             <geometry>
-                <mesh filename="package://minibot_description/meshes/visual/ydlidar_x2_assy.dae" scale="1 1 1"/>
+                <mesh filename="file://$(find minibot_description)/meshes/visual/ydlidar_x2_assy.dae" scale="1 1 1"/>
             </geometry>
         </visual>
@@ -25,5 +25,5 @@
             <origin xyz="0 0 0" rpy="0 0 0"/>
             <geometry>
-                <mesh filename="package://minibot_description/meshes/collision/ydlidar_x2_assy.stl" scale="1 1 1"/>
+                <mesh filename="file://$(find minibot_description)/meshes/collision/ydlidar_x2_assy.stl" scale="1 1 1"/>
             </geometry>
         </collision>
